File: NO2C/vDD1 - SMD/KiCAD/Inputs and Outputs.kicad_sch (KiCad schematic)
At the start: 104 parts, among them IC1 TC4424AVOA, IC2 MPXH6400AC6T1, Q1 NCV8406ASTT3G, Q2 NCV8406ASTT3G, Q3 NCV8406ASTT3G, Q4 NCV8406ASTT3G, Q5 NCV8406ASTT3G, Q6 NCV8406ASTT3G, Q7 AO3400A, U3 MAX9926UAEE+

Commit message: quick parts supply update
Parts:
- C10, C11: LCSC Part C1853786 -> C1636; MPN CC0603JPX7R9BB102 -> 0603CG102J500NT
Changed lines of the file:
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@@
 			)
 		)
-		(property "LCSC Part" "C1853786"
+		(property "LCSC Part" "C1636"
 			(at 359.41 142.24 0)
 			(effects
@@
 			)
 		)
-		(property "MPN" "CC0603JPX7R9BB102"
+		(property "MPN" "0603CG102J500NT"
 			(at 359.41 142.24 0)
 			(effects
@@
 			)
 		)
-		(property "LCSC Part" "C1853786"
+		(property "LCSC Part" "C1636"
 			(at 372.11 142.24 0)
 			(effects
@@
 			)
 		)
-		(property "MPN" "CC0603JPX7R9BB102"
+		(property "MPN" "0603CG102J500NT"
 			(at 372.11 142.24 0)
 			(effects
