File: NO2C/vDD1 - SMD/KiCAD/NO2C.kicad_sch (KiCad schematic)
At the start: 70 parts, among them IC4 CONN_02X08, J1 3-6437285-0, J2 USB_C_Receptacle_USB2.0_16P, P1 Conn_01x04, P4 Conn_01x04, SW1 SW_Push, U1 L7805CDT(UMW), U2 STM32F407VETx, U4 W25Q16JVSS, U5 TJA1050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

Commit message: quick parts supply update
Parts:
- C12, C24: LCSC Part C1853786 -> C1636; MPN CC0603JPX7R9BB102 -> 0603CG102J500NT
Changed lines of the file:
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@@
 			)
 		)
-		(property "LCSC Part" "C1853786"
+		(property "LCSC Part" "C1636"
 			(at 363.22 76.2 0)
 			(effects
@@
 			)
 		)
-		(property "MPN" "CC0603JPX7R9BB102"
+		(property "MPN" "0603CG102J500NT"
 			(at 363.22 76.2 0)
 			(effects
@@
 			)
 		)
-		(property "LCSC Part" "C1853786"
+		(property "LCSC Part" "C1636"
 			(at 311.15 39.37 0)
 			(effects
@@
 			)
 		)
-		(property "MPN" "CC0603JPX7R9BB102"
+		(property "MPN" "0603CG102J500NT"
 			(at 311.15 39.37 0)
 			(effects
