File: NO2C/vDD2 - SMDWB/KICAD/Lambda LSU4.9.kicad_sch (KiCad schematic)
At the start: 21 parts, among them IC3 VNS3NV04DPTR-E, J3 Conn_02x03_Odd_Even, U7 CJ125_32

Commit message: plugin wideband
Added wide band to the main connector.
Parts:
- J3: now left out of the parts list
Changed lines of the file:
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@@
 		(unit 1)
 		(exclude_from_sim no)
-		(in_bom yes)
-		(on_board yes)
+		(in_bom no)
+		(on_board no)
 		(dnp yes)
 		(fields_autoplaced yes)
