File: NO2C/vDD2 - SMDWB/KICAD/NO2C.kicad_sch (KiCad schematic)
At the start: 70 parts, among them IC4 CONN_02X08, J1 3-6437285-0, J2 USB_C_Receptacle_USB2.0_16P, P1 Conn_01x04, P4 Conn_01x04, SW1 SW_Push, U1 L7805CDT(UMW), U2 STM32F407VETx, U4 W25Q16JVSS, U5 TJA1050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

Commit message: plugin wideband
Added wide band to the main connector.
Parts:
- removed R62, R63: 0R, Resistor_SMD:R_0603_1608Metric, symbol Device:R_Small_US
- removed R64, R74: 10K, Resistor_SMD:R_0603_1608Metric, symbol Device:R_Small_US
Connections:
- net GND: no longer J1.21
- net SWCLK: no longer J1.22
- net SWDIO: no longer J1.23
- net IP: now reaches J1.15
- net IA: now reaches J1.16
- new net HEAT-: J1.23
- new net UN: J1.21
- new net VM: J1.22
